File: pcb/sensCorriente.kicad_pcb (KiCad board)
At the start: 2 copper layers, 0 parts

Commit message: Placing de componentes terminado.
Parts:
- added C1: 1uF, C1, F.Cu at (163.8, 169.5)
- added C10: 100nF, C1, F.Cu at (257.8, 153.7)
- added C11: 100nF, C1, F.Cu at (257.8, 161.3)
- added C2: 100nF, C1, F.Cu at (163.8, 173.4)
- added C3: 100nF, C1, F.Cu at (144.8, 148.6)
- added C4: 100nF, C1, F.Cu at (269.9, 121.3)
- added C5: 100nF, C1, F.Cu at (269.2, 183.5)
- added C6: TBD, C1, F.Cu at (269.2, 177.2)
- added C7: 100nF, C1, F.Cu at (260.4, 181.6)
- added C8: 100nF, C1, F.Cu at (257.8, 146.1)
- added C9: 100nF, C1, F.Cu at (269.9, 137.2)
- added J1: I_in, bornier2, F.Cu at (295.3, 180.3)
- added J2: USB, USB_B, F.Cu at (133.3, 145.4)
- added J3: SD-CON, SDCARD-REVERSE, F.Cu at (154.3, 166.4)
- added J4: DB9, DB9_SHIELD, F.Cu at (283.8, 153.0)
- added P1: LPCXpresso, LPCXpresso, F.Cu at (211.5, 172.1)
- added R1: 10k, R3, F.Cu at (164.5, 180.3)
- added R2: 10k, R3, F.Cu at (164.5, 176.5)
- added R3: 10k, R3, F.Cu at (164.5, 166.4)
- added R4: 10k, R3, F.Cu at (164.5, 162.6)
- added R5: 10k, R3, F.Cu at (164.5, 184.2)
- added R6: 10k, R3, F.Cu at (164.5, 158.8)
- added R7: 10k, R3, F.Cu at (268.6, 180.3)
- added R8: 100, R3, F.Cu at (233.0, 128.3)
- added RV1: POT, RV2X4, F.Cu at (258.4, 124.5)
- added S1: Display 16x2, Display16x2, F.Cu at (174.0, 119.4)
- added SW1: CALIB, SW_PUSH_SMALL, F.Cu at (276.9, 120.7)
- added U1: ACS713, SO8E, F.Cu at (281.3, 180.3)
- added U2: MAX232, DIP-16__300_ELL, F.Cu at (269.9, 153.7)
