File: pcb/sensCorriente.kicad_pcb (KiCad board)
At the start: 2 copper layers, 29 parts, among them J1 I_in, J2 USB, J3 SD-CON, J4 DB9, P1 LPCXpresso, SW1 CALIB, U1 ACS713, U2 MAX232

Commit message: Avance en el trazado de vias.
Routing:
- net +5V: track 0.00 -> 212.9 mm, vias 0 -> 3
- net /LCD_RS: track 0.00 -> 76.8 mm
- net /USB_D+: track 0.00 -> 74.7 mm
- net /LCD_E: track 0.00 -> 72.8 mm
- net /LCD_D7: track 0.00 -> 70.2 mm
- net /LCD_D4: track 0.00 -> 69.5 mm
- net /LCD_D5: track 0.00 -> 67.6 mm
- net /USB_D-: track 0.00 -> 67.5 mm
- net /LCD_D6: track 0.00 -> 66.5 mm
- net +3.3V: track 0.00 -> 55.7 mm
- net /SD_SSEL: track 0.00 -> 54.0 mm, vias 0 -> 2
- net /SD_CLK: track 0.00 -> 44.8 mm, vias 0 -> 2
- net /SD_MISO: track 0.00 -> 44.4 mm, vias 0 -> 2
- net /SD_MOSI: track 0.00 -> 43.6 mm, vias 0 -> 2
- net N-0000047: track 0.00 -> 18.7 mm, vias 0 -> 2
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
Commit message: Trazado preliminar
Routing:
- net N-0000039: track 0.00 -> 103.2 mm
- net /TXD1: track 0.00 -> 87.7 mm, vias 0 -> 2
- net /RXD1: track 0.00 -> 83.6 mm, vias 0 -> 2
- net /CTS1: track 0.00 -> 78.8 mm, vias 0 -> 2
- net /CALIB: track 11.1 -> 88.9 mm
- net /RTS1: track 0.00 -> 63.7 mm, vias 0 -> 2
- net /AIN0: track 4.44 -> 58.7 mm
- net N-0000080: track 0.00 -> 47.6 mm
- net +5V: track 212.9 -> 255.8 mm
- net N-0000034: track 0.00 -> 29.1 mm
- net N-0000035: track 0.00 -> 22.8 mm
- net /SD_MISO: track 44.4 -> 40.4 mm
- net +3.3V: track 55.7 -> 52.0 mm
- net /USB_D+: track 74.7 -> 77.8 mm
- net /SD_SSEL: track 54.0 -> 52.9 mm
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